File: rSTM32F405RGT6_B/rSTM32F405RGT6_B.kicad_pcb (KiCad board)
At the start: 2 copper layers, 42.2 x 55.8 mm, 53 parts, among them J1 USB, J2 BOOT, J3 STLink, J4 , J5 , J6 , SW1 RESET, U1 STM32F405RGT6, U2 RT9013, U3 MP2359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

Commit message: KiCAD Project
Fixing some footprints.
Parts:
- SW1: footprint Buttons_Switches_SMD:SW_SPST_EVPBF -> .rpvM:Switch_SMD_5.2x6.4_reset
Changed lines of the file:
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@@
       (effects (font (size 1 1) (thickness 0.15)) (justify mirror))
     )
+    (fp_line (start -1.9 2) (end 1.9 2) (layer B.SilkS) (width 0.15))
+    (fp_line (start -1.9 -2) (end 1.9 -2) (layer B.SilkS) (width 0.15))
+    (fp_line (start 4 -2) (end 3.6 -2) (layer B.SilkS) (width 0.15))
+    (fp_line (start 4 2) (end 3.6 2) (layer B.SilkS) (width 0.15))
+    (fp_line (start -4 2) (end -3.6 2) (layer B.SilkS) (width 0.15))
+    (fp_line (start -4 -2) (end -3.6 -2) (layer B.SilkS) (width 0.15))
     (fp_arc (start -4 0) (end -4 -0.6) (angle 180) (layer B.SilkS) (width 0.15))
     (fp_circle (center 3.1 0) (end 3.5 -0.1) (layer B.SilkS) (width 0.15))
     (fp_line (start -4 -2) (end -4 2) (layer B.SilkS) (width 0.15))
-    (fp_line (start 4 -2) (end -4 -2) (layer B.SilkS) (width 0.15))
     (fp_line (start 4 2) (end 4 -2) (layer B.SilkS) (width 0.15))
-    (fp_line (start -4 2) (end 4 2) (layer B.SilkS) (width 0.15))
     (pad 4 smd rect (at -2.75 1.6) (size 1.3 1.9) (layers B.Cu B.Paste B.Mask)
       (net 9 /PC15))
@@
     (pad 1 smd rect (at -2.75 -1.6) (size 1.3 1.9) (layers B.Cu B.Paste B.Mask)
       (net 8 /PC14))
+  )
+  (module .rpvM:Switch_SMD_5.2x6.4_reset (layer F.Cu)
+    (at 70 60.7 90)
+    (fp_text reference SW1 (at -3.1 4.1 90) (layer F.SilkS)
+      (effects (font (size 1 1) (thickness 0.15)))
+    )
+    (fp_text value RESET (at 2.3 4.2 90) (layer F.Fab)
+      (effects (font (size 1 1) (thickness 0.15)))
+    )
+    (fp_line (start -2.2 -1) (end -1.6 -2.3) (layer F.SilkS) (width 0.15))
+    (fp_line (start -1.5 2.3) (end -2.2 1) (layer F.SilkS) (width 0.15))
+    (fp_line (start 1.4 2.3) (end 2.1 1.2) (layer F.SilkS) (width 0.15))
+    (fp_line (start 2.1 -1) (end 1.4 -2.3) (layer F.SilkS) (width 0.15))
+    (fp_line (start -1.6 -2.3) (end 1.4 -2.3) (layer F.SilkS) (width 0.15))
+    (fp_line (start 2.1 1.2) (end 2.1 -1) (layer F.SilkS) (width 0.15))
+    (fp_line (start -1.5 2.3) (end 1.4 2.3) (layer F.SilkS) (width 0.15))
+    (fp_line (start -2.2 -1) (end -2.2 1) (layer F.SilkS) (width 0.15))
+    (fp_text user %R (at -3.1 4.1 90) (layer F.Fab)
+      (effects (font (size 1 1) (thickness 0.15)))
+    )
+    (pad 1 smd rect (at 3.1 -1.85 90) (size 1.8 1.1) (layers F.Cu F.Paste F.Mask)
+      (net 7 /NRST))
+    (pad 2 smd rect (at 3.1 1.85 90) (size 1.8 1.1) (layers F.Cu F.Paste F.Mask)
+      (net 2 GND))
+    (pad 2 smd rect (at -3.1 1.85 90) (size 1.8 1.1) (layers F.Cu F.Paste F.Mask)
+      (net 2 GND))
+    (pad 1 smd rect (at -3.1 -1.85 90) (size 1.8 1.1) (layers F.Cu F.Paste F.Mask)
+      (net 7 /NRST))
   )
   (module Capacitors_SMD:C_0805 (layer B.Cu)
@@
       (at (xyz 0 0 0))
       (scale (xyz 1 1 1))
-      (rotate (xyz 0 0 0))
-    )
-  )
-  (module Buttons_Switches_SMD:SW_SPST_EVPBF (layer F.Cu)
-    (at 70 60.7 90)
-    (descr "Light Touch Switch")
-    (attr smd)
-    (fp_text reference SW1 (at -3.1 4.1 90) (layer F.SilkS)
-      (effects (font (size 1 1) (thickness 0.15)))
-    )
-    (fp_text value RESET (at 2.3 4.2 90) (layer F.Fab)
-      (effects (font (size 1 1) (thickness 0.15)))
-    )
-    (fp_circle (center 0 0) (end 1.7 0) (layer F.Fab) (width 0.1))
-    (fp_line (start -4.5 3.25) (end -4.5 -3.25) (layer F.CrtYd) (width 0.05))
-    (fp_line (start 4.5 3.25) (end -4.5 3.25) (layer F.CrtYd) (width 0.05))
-    (fp_line (start 4.5 -3.25) (end 4.5 3.25) (layer F.CrtYd) (width 0.05))
-    (fp_line (start -4.5 -3.25) (end 4.5 -3.25) (layer F.CrtYd) (width 0.05))
-    (fp_text user %R (at -3.1 4.1 90) (layer F.Fab)
-      (effects (font (size 1 1) (thickness 0.15)))
-    )
-    (fp_line (start -3 3) (end -3 -3) (layer F.Fab) (width 0.1))
-    (fp_line (start 3 3) (end -3 3) (layer F.Fab) (width 0.1))
-    (fp_line (start 3 -3) (end 3 3) (layer F.Fab) (width 0.1))
-    (fp_line (start -3 -3) (end 3 -3) (layer F.Fab) (width 0.1))
-    (fp_line (start -3.15 -2.65) (end -3.15 -3.1) (layer F.SilkS) (width 0.12))
-    (fp_line (start 3.15 -3.1) (end 3.15 -2.65) (layer F.SilkS) (width 0.12))
-    (fp_line (start -3.15 -3.1) (end 3.15 -3.1) (layer F.SilkS) (width 0.12))
-    (fp_line (start 3.15 -1.35) (end 3.15 1.35) (layer F.SilkS) (width 0.12))
-    (fp_line (start -3.15 1.35) (end -3.15 -1.35) (layer F.SilkS) (width 0.12))
-    (fp_line (start 3.15 3.1) (end 3.15 2.7) (layer F.SilkS) (width 0.12))
-    (fp_line (start -3.15 3.1) (end 3.15 3.1) (layer F.SilkS) (width 0.12))
-    (fp_line (start -3.15 2.65) (end -3.15 3.1) (layer F.SilkS) (width 0.12))
-    (pad 2 smd rect (at 2.88 2 90) (size 2.75 1) (layers F.Cu F.Paste F.Mask)
-      (net 2 GND))
-    (pad 2 smd rect (at -2.88 2 90) (size 2.75 1) (layers F.Cu F.Paste F.Mask)
-      (net 2 GND))
-    (pad 1 smd rect (at -2.88 -2 90) (size 2.75 1) (layers F.Cu F.Paste F.Mask)
-      (net 7 /NRST))
-    (pad 1 smd rect (at 2.88 -2 90) (size 2.75 1) (layers F.Cu F.Paste F.Mask)
-      (net 7 /NRST))
-    (model ${KISYS3DMOD}/Buttons_Switches_SMD.3dshapes/SW_SPST_EVPBF.wrl
-      (at (xyz 0 0 0))
-      (scale (xyz 1 1 1))
