File: rSTM32F405RGT6_B/rSTM32F405RGT6_B.sch (KiCad schematic (older format))
At the start: 37 parts, among them J1 USB, J2 BOOT, J3 STLink, J4 , J5 , J6 , SW1 RESET, U1 STM32F405RGT6, Y1 CSTCE8.000M, Y2 32.768K

Commit message: KiCAD Project
Fixing some footprints.
Parts:
- SW1: footprint Buttons_Switches_SMD:SW_SPST_EVPBF -> .rpvM:Switch_SMD_5.2x6.4_reset
Changed lines of the file:
@@
 F 0 "SW1" H 3550 2950 50  0000 L CNN
 F 1 "RESET" H 3800 2950 50  0000 L CNN
-F 2 "Buttons_Switches_SMD:SW_SPST_EVPBF" H 3750 3000 50  0001 C CNN
+F 2 ".rpvM:Switch_SMD_5.2x6.4_reset" H 3750 3000 50  0001 C CNN
 F 3 "~" H 3750 3000 50  0001 C CNN
 	1    3750 2800
